File: RPi_Teleco_PCB/RPi_Teleco_PCB.sch (KiCad schematic (older format))
At the start: 14 parts, among them U1 MCP23017_SP

Commit message: top
Parts:
- added R1, R2: 4.7k, Resistor_THT:R_Axial_DIN0207_L6.3mm_D2.5mm_P7.62mm_Horizontal, symbol Device:R
Connections:
- net +5V: now also R1.1, R2.1
- net GND: now also U1.15 (A0), U1.16 (A1), U1.17 (A2)
- net SCK: now also R2.2
- net SDA: now also R1.2
Other:
- note added: "PULL-UP I2C"
- note added: "Pinout order\nà confirmer"
- note removed: "Confirmer Connections \nVDD = VCC\nVSS = GND"
- moved on the sheet: 5V-GND1, Input1, Power_Switch1A, Rpi-Power1, Screen1, Switch1, Switch2, Switch3, Switch4, Switch5, Switch6, Switch7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
