File: RPi_Teleco_PCB/RPi_Teleco_PCB.kicad_pcb (KiCad board)
At the start: 2 copper layers, 14 parts, among them U1 MCP23017_SP

Commit message: y
Parts:
- moved U1 1.27 mm to (91.4, 78.7)
Changed lines of the file:
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@@
       (effects (font (size 0.6096 0.6096) (thickness 0.127)))
     )
-    (fp_text value MOMENTARY-SWITCH-SPST-LED-PTH-12MM (at 3.175 6.731) (layer F.SilkS)
+    (fp_text value MOMENTARY-SWITCH-SPST-LED-PTH-12MM (at 3.175 6.731) (layer F.SilkS) hide
       (effects (font (size 0.6096 0.6096) (thickness 0.127)))
     )
@@
       (effects (font (size 0.6096 0.6096) (thickness 0.127)))
     )
-    (fp_text value MOMENTARY-SWITCH-SPST-LED-PTH-12MM (at 3.175 6.731) (layer F.SilkS)
+    (fp_text value MOMENTARY-SWITCH-SPST-LED-PTH-12MM (at 3.175 6.731) (layer F.SilkS) hide
       (effects (font (size 0.6096 0.6096) (thickness 0.127)))
     )
@@
       (effects (font (size 0.6096 0.6096) (thickness 0.127)))
     )
-    (fp_text value MOMENTARY-SWITCH-SPST-LED-PTH-12MM (at 3.175 6.731) (layer F.SilkS)
+    (fp_text value MOMENTARY-SWITCH-SPST-LED-PTH-12MM (at 3.175 6.731) (layer F.SilkS) hide
       (effects (font (size 0.6096 0.6096) (thickness 0.127)))
     )
@@
       (effects (font (size 0.6096 0.6096) (thickness 0.127)))
     )
-    (fp_text value MOMENTARY-SWITCH-SPST-LED-PTH-12MM (at 3.175 6.731) (layer F.SilkS)
+    (fp_text value MOMENTARY-SWITCH-SPST-LED-PTH-12MM (at 3.175 6.731) (layer F.SilkS) hide
       (effects (font (size 0.6096 0.6096) (thickness 0.127)))
     )
@@
       (effects (font (size 0.6096 0.6096) (thickness 0.127)))
     )
-    (fp_text value MOMENTARY-SWITCH-SPST-LED-PTH-12MM (at 3.175 6.731) (layer F.SilkS)
+    (fp_text value MOMENTARY-SWITCH-SPST-LED-PTH-12MM (at 3.175 6.731) (layer F.SilkS) hide
       (effects (font (size 0.6096 0.6096) (thickness 0.127)))
     )
@@
       (effects (font (size 0.6096 0.6096) (thickness 0.127)))
     )
-    (fp_text value MOMENTARY-SWITCH-SPST-LED-PTH-12MM (at 3.175 6.731) (layer F.SilkS)
+    (fp_text value MOMENTARY-SWITCH-SPST-LED-PTH-12MM (at 3.175 6.731) (layer F.SilkS) hide
       (effects (font (size 0.6096 0.6096) (thickness 0.127)))
     )
@@
       (effects (font (size 0.6096 0.6096) (thickness 0.127)))
     )
-    (fp_text value MOMENTARY-SWITCH-SPST-LED-PTH-12MM (at 3.175 6.731) (layer F.SilkS)
+    (fp_text value MOMENTARY-SWITCH-SPST-LED-PTH-12MM (at 3.175 6.731) (layer F.SilkS) hide
       (effects (font (size 0.6096 0.6096) (thickness 0.127)))
     )
@@
       (effects (font (size 0.6096 0.6096) (thickness 0.127)))
     )
-    (fp_text value MOMENTARY-SWITCH-SPST-LED-PTH-12MM (at 3.175 6.731) (layer F.SilkS)
+    (fp_text value MOMENTARY-SWITCH-SPST-LED-PTH-12MM (at 3.175 6.731) (layer F.SilkS) hide
       (effects (font (size 0.6096 0.6096) (thickness 0.127)))
     )
@@
   )
   (module Package_DIP:DIP-28_W7.62mm (layer F.Cu)
-    (at 92.71 78.74 90)
+    (at 91.44 78.74 90)
     (descr "28-lead though-hole mounted DIP package, row spacing 7.62 mm (300 mils)")
     (tags "THT DIP DIL PDIP 2.54mm 7.62mm 300mil")

Commit message: top
Parts:
- added R1: 4.7k, Resistor_THT:R_Axial_DIN0207_L6.3mm_D2.5mm_P7.62mm_Horizontal, F.Cu at (93.8, 94.2)
- added R2: 4.7k, Resistor_THT:R_Axial_DIN0207_L6.3mm_D2.5mm_P7.62mm_Horizontal, F.Cu at (93.8, 98.3)
- moved Rpi-Power1 40.5 mm to (237.5, 95.2)
- moved Power_Switch1 40.5 mm to (252.7, 92.7)
- moved Switch1 39.4 mm to (114.3, 81.3)
- moved Switch3 39.4 mm to (146.4, 81.3)
- moved Switch4 39.4 mm to (162.6, 81.3)
- moved Switch7 39.4 mm to (210.8, 81.2)
- moved Switch8 39.4 mm to (226.4, 81.2)
- moved Switch2 39.4 mm to (130.3, 81.2)
- moved Switch5 39.4 mm to (179.0, 81.2)
- moved Switch6 39.4 mm to (194.7, 81.2)
- moved 5V-GND1 38.4 mm to (262.9, 92.7)
- moved U1 28.0 mm to (109.2, 100.3)
- moved Screen1 15.5 mm to (114.3, 53.3)
- moved Input1 13.0 mm to (95.2, 43.2)
Connections:
- U1 pad 15: Net-(U1-Pad15) -> GND
- U1 pad 16: Net-(U1-Pad16) -> GND
- U1 pad 17: Net-(U1-Pad17) -> GND
Other:
- board text added: "SCREEN"

Commit message: ok
Parts:
- removed 5V-GND1: Screw_Terminal_01x02, TerminalBlock:TerminalBlock_bornier-2_P5.08mm
- removed Input1: From_RPI, Connector_PinSocket_2.54mm:PinSocket_1x04_P2.54mm_Vertical
- removed Power_Switch1: SW, Connector_PinHeader_2.54mm:PinHeader_1x03_P2.54mm_Vertical
- removed R1, R2: 4.7k, Resistor_THT:R_Axial_DIN0207_L6.3mm_D2.5mm_P7.62mm_Horizontal
- removed Rpi-Power1: Conn_01x02_Female, Connector_PinSocket_2.54mm:PinSocket_1x02_P2.54mm_Vertical
- removed Screen1: SPI, Connector_PinSocket_2.54mm:PinSocket_1x04_P2.54mm_Vertical
- added B1: ARDUINO_PRO_MICRO, SPARKFUN_PRO_MICRO, B.Cu at (132.1, 85.1)
- added J1: Conn_01x07, Connector_PinHeader_2.54mm:PinHeader_1x07_P2.54mm_Vertical, F.Cu at (188.0, 65.2)
- added M3: MountingHole_3.2mm_M3, MountingHole:MountingHole_3.2mm_M3, F.Cu at (124.5, 48.3)
- added M3: MountingHole_3.2mm_M3, MountingHole:MountingHole_3.2mm_M3, F.Cu at (124.5, 119.4)
- added M3: MountingHole_3.2mm_M3, MountingHole:MountingHole_3.2mm_M3, F.Cu at (231.1, 119.4)
- added M3: MountingHole_3.2mm_M3, MountingHole:MountingHole_3.2mm_M3, F.Cu at (231.1, 48.3)
- added M3: MountingHole_3.2mm_M3, MountingHole:MountingHole_3.2mm_M3, F.Cu at (146.6, 104.9)
- added M3: MountingHole_3.2mm_M3, MountingHole:MountingHole_3.2mm_M3, F.Cu at (214.1, 104.9)
- added Q1: PN2222A, Package_TO_SOT_THT:TO-92_Inline, F.Cu at (130.8, 106.7)
- Switch1, Switch2, Switch3, Switch4, Switch5, Switch6, Switch7, Switch8: footprint TACTILE_SWITCH_LED_PTH_12MM -> Switches:TACTILE_SWITCH_LED_PTH_12MM
- moved U1 86.4 mm to (179.1, 49.5), turned to 270 degrees
- moved Switch4 56.4 mm to (207.0, 116.0)
- moved Switch3 55.1 mm to (189.2, 116.0)
- moved Switch2 53.8 mm to (171.4, 116.0)
- moved Switch1 52.5 mm to (153.7, 116.0)
- moved Switch6 30.8 mm to (207.0, 53.0)
- moved Switch5 30.1 mm to (189.2, 53.0)
- moved Switch7 15.8 mm to (226.1, 77.5)
- moved Switch8 14.5 mm to (226.1, 95.8)
Connections:
- Switch1 pad A: LED1 -> Level
- Switch1 pad C: GND -> LED1
- Switch2 pad A: LED2 -> Level
- Switch2 pad C: GND -> LED2
- Switch3 pad A: LED3 -> Level
- Switch3 pad C: GND -> LED3
- Switch4 pad A: LED4 -> Level
- Switch4 pad C: GND -> LED4
- Switch5 pad A: LED5 -> Level
- Switch5 pad C: GND -> LED5
- Switch6 pad A: LED6 -> Level
- Switch6 pad C: GND -> LED6
- Switch7 pad A: LED7 -> Level
- Switch7 pad C: GND -> LED7
- Switch8 pad A: LED8 -> Level
- Switch8 pad C: GND -> LED8
- U1 pad 11: Net-(U1-Pad11) -> (no net)
- U1 pad 12: SCK -> I2C_SCL
- U1 pad 13: SDA -> I2C_SDA
- U1 pad 14: Net-(U1-Pad14) -> (no net)
- U1 pad 18: Net-(U1-Pad18) -> +5V
- U1 pad 19: Net-(U1-Pad19) -> (no net)
- U1 pad 2: BTN2 -> LED1
- U1 pad 20: Net-(U1-Pad20) -> (no net)
- U1 pad 21: LED1 -> BTN5
- U1 pad 22: LED2 -> LED5
- U1 pad 23: LED3 -> BTN6
- U1 pad 24: LED4 -> LED6
- U1 pad 25: LED5 -> BTN7
- U1 pad 26: LED6 -> LED7
- U1 pad 27: LED7 -> BTN8
- U1 pad 3: BTN3 -> BTN2
- U1 pad 4: BTN4 -> LED2
- U1 pad 5: BTN5 -> BTN3
- U1 pad 6: BTN6 -> LED3
- U1 pad 7: BTN7 -> BTN4
- U1 pad 8: BTN8 -> LED4
Other:
- board outline added: 116.8 x 81.3 mm
- board text added: "2.42’’ OLED DISPLAY"
- board text added: "RPi-Teleco KXKM 2020"
- board text added: "USB"
- board text removed: "SCREEN"

Commit message: ready
Parts:
- removed the M3 at (124.5, 48.3)
- removed the M3 at (231.1, 48.3)
- added M3: MountingHole_3.2mm_M3, MountingHole:MountingHole_3.2mm_M3, F.Cu at (125.7, 50.8)
- added M3: MountingHole_3.2mm_M3, MountingHole:MountingHole_3.2mm_M3, F.Cu at (229.9, 50.8)
- moved U1 36.4 mm to (143.5, 57.1), turned to 90 degrees
- moved Q1 2.54 mm to (133.3, 106.7), turned to 180 degrees
- moved M3 1.27 mm to (125.7, 119.4)
- moved Switch5 1.27 mm to (189.2, 54.2)
- moved Switch6 1.27 mm to (207.0, 54.2)
- moved M3 1.27 mm to (229.9, 119.4)
Routing:
- net Level: track 0.00 -> 259.4 mm
- net LED7: track 0.00 -> 152.3 mm, vias 0 -> 1
- net LED8: track 0.00 -> 126.1 mm
- net +5V: track 0.00 -> 115.1 mm
- net BTN8: track 0.00 -> 108.2 mm
- net BTN7: track 0.00 -> 97.3 mm
- net BTN4: track 0.00 -> 91.6 mm, vias 0 -> 1
- net LED4: track 0.00 -> 85.3 mm, vias 0 -> 1
- net BTN3: track 0.00 -> 84.4 mm, vias 0 -> 1
- net LED3: track 0.00 -> 80.2 mm, vias 0 -> 1
- net LED2: track 0.00 -> 75.0 mm, vias 0 -> 1
- net BTN2: track 0.00 -> 74.5 mm, vias 0 -> 1
- net SCK: track 0.00 -> 73.3 mm
- net SDA: track 0.00 -> 70.4 mm
- net LED1: track 0.00 -> 69.8 mm, vias 0 -> 1
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- added copper zone on B.Cu, net GND
Other:
- board size 116.8 x 81.3 mm -> 114.3 x 78.7 mm
